File: kicad/nrf.kicad_pcb (KiCad board)
At the start: 2 copper layers, 17.8 x 38.1 mm, 6 parts, among them P1 ICSP, P2 CONN_01X02, P3 NRF_24L01, U1 MCP1755ST-3302E/DB

Commit message: Voltage regulator
Parts:
- added C3: 10uF, Capacitors_SMD:C_0805_HandSoldering, F.Cu at (158.7, 89.8)
- added C4: 10uF, Capacitors_SMD:C_0805_HandSoldering, F.Cu at (157.9, 100.9)
- C1, C2: moved to B.Cu
- P3: footprint Socket_Strips:Socket_Strip_Straight_2x04 -> NRF_24L01
- U1: value MCP1755ST-3302E/DB -> MCP1700_SOT-89; footprint TO_SOT_Packages_SMD:SOT-223 -> TO_SOT_Packages_SMD:SOT89-3_Housing_Handsoldering; moved to B.Cu
- moved C2 46.0 mm to (159.2, 89.8), turned to 270 degrees
- moved C1 45.6 mm to (169.6, 90.0), turned to 90 degrees
- moved U1 21.0 mm to (164.2, 89.8), turned to 90 degrees
- moved P1 10.7 mm to (161.2, 102.5)
- moved P3 4.66 mm to (162.5, 93.6)
- moved P2 2.55 mm to (163.7, 105.0)
Connections:
- U1 pad 1: 5V -> GND
- U1 pad 2: GND -> 5V
Other:
- board size 17.8 x 38.1 mm -> 15.2 x 20.3 mm

Commit message: Traces
Parts:
- C4: moved to B.Cu
- moved C4 11.8 mm to (169.6, 99.5)
- moved P2 2.69 mm to (166.4, 105.3), turned to 180 degrees
- moved C3 1.28 mm to (159.9, 90.0), turned to 0 degrees
- moved C1 0.76 mm to (169.6, 90.8)
Connections:
- P1 pad 5: (no net) -> Net-(P1-Pad5)
- P2 pad 1: (no net) -> CSN
- P2 pad 2: (no net) -> CE
- P3 pad 3: (no net) -> CE
- P3 pad 4: (no net) -> CSN
- P3 pad 8: (no net) -> Net-(P3-Pad8)
Routing:
- net GND: track 0.00 -> 76.5 mm
- net 5V: track 0.00 -> 25.5 mm
- net CSN: track 0.00 -> 20.9 mm
- net CE: track 0.00 -> 13.0 mm
- net 3V3: track 0.00 -> 12.8 mm
- net MISO: track 0.00 -> 12.1 mm
- net MOSI: track 0.00 -> 7.48 mm
- net SCK: track 0.00 -> 7.48 mm
- added copper zone on B.Cu, net GND
- added copper zone on F.Cu, net GND
Other:
- net class Default: clearance 0.3048 -> 0.2286
- net class wide added: clearance 0.3556, trace_width 0.4064, via_dia 0.8128, via_drill 0.4064
- rule trace_clearance: 0.3048 -> 0.2286

Commit message: Logo
Parts:
- added REF**: TheApiLogoTiny, nrf:TheApiLogoTiny, F.Cu at (158.3, 102.2)
- moved C3 0.52 mm to (159.8, 89.5)
Other:
- board text added: "."
- board text added: "CE"
- board text added: "CSN"
- board text added: "petermclarke@gmail.com"
